File: ScintillatorProbeHardware/ScintillatorProbeHardware.kicad_sch (KiCad schematic)
At the start: 112 parts, among them J1 USB_B, J2 Conn_01x02, J3 Conn_01x03, J4 Conn_01x04, J7 Conn_01x02, J8 Conn_01x03, J9 Conn_01x01, Q1 15N10, Q2 S8050, Q3 S8050, Q4 AO401, Q5 S8050, Q6 S8050, Q7 S8050, T1 24:1800, U1 ICL7660, U3 LM358, U4 STM32F103C8Tx, U5 USBLC6-2SC6, U6 AMS1117-3.3, U7 LM318N, U8 LM318N, U9 LM318N, Y1 32.768kHz, Y2 8MHz

Commit message: Hardware finisnig touches, Software directory typo fixed
Parts:
- added J10: Conn_01x04, Connector_PinHeader_2.54mm:PinHeader_1x04_P2.54mm_Vertical, symbol Connector_Generic:Conn_01x04
Connections:
- net +5V: now also J10.1 (Pin_1)
- net GND: now also J10.4 (Pin_4)
- net UART_TX: now reaches U4.30 (PA9)
- net UART_TX: now also J10.2 (Pin_2)
- net UART_RX: now reaches U4.31 (PA10)
- net UART_RX: now also J10.3 (Pin_3)
Other:
- note added: "OP Amp voltage supply"
- note added: "PMT signal aplifier and sample & hold circuit"
- note removed: "OPAmp voltage supply"
- note removed: "PMT signal aplifier, trigger and sample & hold circuit"

Commit message: Hardware revision 1 as sent to manifacture
Parts:
- removed Q4: AO401, Package_TO_SOT_SMD:SOT-23, symbol Simulation_SPICE:PMOS
- removed U5: USBLC6-2SC6, Package_TO_SOT_SMD:SOT-23-6, symbol Power_Protection:USBLC6-2SC6
- added C33, C34, C35, C36, C37, C38: 1u, Capacitor_SMD:C_0603_1608Metric, symbol Device:C
- added Q8: MDD2302, Package_TO_SOT_SMD:SOT-23, symbol Device:Q_NMOS_GSD
- added R40: 1k, Resistor_SMD:R_0603_1608Metric, symbol Device:R
- added SYM1, SYM2, SYM3, SYM4, SYM5, SYM6: SYM_Flash_Small, CustomParts:W012 - electricity hazard, symbol Graphic:SYM_Flash_Small
- C12, C18, C26: LCSC https://www.lcsc.com/product-detail/Multilayer-Ceramic-Capa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 -> C6119867; LCSC Part Number C6119867 -> (none); LCSC URL (none) -> https://www.lcsc.com/product-detail/Multilayer-Ceramic-Capa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
- C13, C17, C27, C28, C29, C30, C31, C32: LCSC https://www.lcsc.com/product-detail/Multilayer-Ceramic-Capa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 -> C15849; LCSC Part Number C15849 -> (none); LCSC URL (none) -> https://www.lcsc.com/product-detail/Multilayer-Ceramic-Capa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
- C16: LCSC https://www.lcsc.com/product-detail/Aluminum-Electrolytic-C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 -> C5162355; LCSC Part Number C5162355 -> (none); LCSC URL (none) -> https://www.lcsc.com/product-detail/Aluminum-Electrolytic-C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
- C19, C2, C20, C21, C3, C6, C7: LCSC https://www.lcsc.com/product-detail/Aluminum-Electrolytic-C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 -> RVT1V100M0405; LCSC Part Number RVT1V100M0405 -> (none); LCSC URL (none) -> https://www.lcsc.com/product-detail/Aluminum-Electrolytic-C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
- C22, C23, C24, C25: LCSC https://www.lcsc.com/product-detail/Multilayer-Ceramic-Capa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 -> C1648; LCSC Part Number C105621 -> (none); LCSC URL (none) -> https://www.lcsc.com/product-detail/Multilayer-Ceramic-Capa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
- C4: LCSC https://www.lcsc.com/product-detail/Aluminum-Electrolytic-C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 -> C5162355; LCSC Part Number C5162355 -> (none); LCSC URL (none) -> https://www.lcsc.com/product-detail/Aluminum-Electrolytic-C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; TME (none) -> https://www.tme.eu/cz/details/vb1c102mg105000ce0/elektrolyt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
- C5: LCSC https://www.lcsc.com/product-detail/Multilayer-Ceramic-Capa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 -> C15850; LCSC Part Number C1713 -> (none); LCSC URL (none) -> https://www.lcsc.com/product-detail/Multilayer-Ceramic-Capa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
- C8: LCSC https://www.lcsc.com/product-detail/Multilayer-Ceramic-Capa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 -> C1525; LCSC Part Number C14663 -> (none); LCSC URL (none) -> https://www.lcsc.com/product-detail/Multilayer-Ceramic-Capa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
- D2, D3, D5, D6: LCSC https://www.lcsc.com/product-detail/Schottky-Diodes_onsemi-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 -> C7502702; LCSC Part Number C145179 -> (none); LCSC URL (none) -> https://www.lcsc.com/product-detail/Schottky-Diodes_onsemi-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
- FB1, FB2, FB3, FB4: LCSC https://www.lcsc.com/product-detail/Ferrite-Beads_Murata-El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 -> C2661807; LCSC Part Number C2661807 -> (none); LCSC URL (none) -> https://www.lcsc.com/product-detail/Ferrite-Beads_Murata-El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
- Q1: LCSC https://www.lcsc.com/product-detail/MOSFETs_UMW-Youtai-Semi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 -> C359106; LCSC Part Number C359106 -> (none); LCSC URL (none) -> https://www.lcsc.com/product-detail/MOSFETs_UMW-Youtai-Semi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
- Q2, Q3, Q5, Q6, Q7: LCSC https://www.lcsc.com/product-detail/Bipolar-BJT_Guangdong-H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 -> C2146; LCSC Part Number C181158 -> (none); LCSC URL (none) -> https://www.lcsc.com/product-detail/Bipolar-BJT_Guangdong-H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
- R1, R2: LCSC https://www.lcsc.com/product-detail/Chip-Resistor-Surface-M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 -> C3014189; LCSC Part Number C3014189 -> (none); LCSC URL (none) -> https://www.lcsc.com/product-detail/Chip-Resistor-Surface-M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
- R10, R11, R12, R13, R14, R15, R16, R17, R18, R6, R9: LCSC https://www.lcsc.com/product-detail/Chip-Resistor-Surface-M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 -> C2907378; LCSC Part Number C2907378 -> (none); LCSC URL (none) -> https://www.lcsc.com/product-detail/Chip-Resistor-Surface-M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
- R19, R35, R36, R38, R39, R8: LCSC https://www.lcsc.com/product-detail/Chip-Resistor-Surface-M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 -> C21190; LCSC Part Number C21190 -> (none); LCSC URL (none) -> https://www.lcsc.com/product-detail/Chip-Resistor-Surface-M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
- R20, R5: LCSC https://www.lcsc.com/product-detail/Chip-Resistor-Surface-M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 -> C25804; LCSC Part Number C25804 -> (none); LCSC URL (none) -> https://www.lcsc.com/product-detail/Chip-Resistor-Surface-M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
- R21, R23: footprint Resistor_SMD:R_1812_4532Metric -> Resistor_SMD:R_0603_1608Metric; LCSC https://www.lcsc.com/product-detail/Chip-Resistor-Surface-M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 -> C23138; LCSC Part Number C2933950 -> (none); LCSC URL (none) -> https://www.lcsc.com/product-detail/Chip-Resistor-Surface-M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
- R22, R3: LCSC https://www.lcsc.com/product-detail/Chip-Resistor-Surface-M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 -> C17713; LCSC Part Number C102018 -> (none); LCSC URL (none) -> https://www.lcsc.com/product-detail/Chip-Resistor-Surface-M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
- R24: LCSC https://www.lcsc.com/product-detail/Chip-Resistor-Surface-M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 -> C23260; LCSC Part Number C23260 -> (none); LCSC URL (none) -> https://www.lcsc.com/product-detail/Chip-Resistor-Surface-M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
- R25, R26, R27, R28, R31, R32, R33, R34: LCSC https://www.lcsc.com/product-detail/Chip-Resistor-Surface-M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 -> C2075184; LCSC Part Number C2075184 -> (none); LCSC URL (none) -> https://www.lcsc.com/product-detail/Chip-Resistor-Surface-M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
- R29: LCSC https://www.lcsc.com/product-detail/Chip-Resistor-Surface-M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 -> 0603; LCSC Part Number 0603 -> (none); LCSC URL (none) -> https://www.lcsc.com/product-detail/Chip-Resistor-Surface-M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
- R30: footprint Resistor_SMD:R_2010_5025Metric -> Resistor_SMD:R_0805_2012Metric; LCSC https://www.lcsc.com/product-detail/Chip-Resistor-Surface-M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 -> C17714; LCSC Part Number C2960940 -> (none); LCSC URL (none) -> https://www.lcsc.com/product-detail/Chip-Resistor-Surface-M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
- R37, R4: footprint Resistor_SMD:R_1812_4532Metric -> Resistor_SMD:R_2010_5025Metric; LCSC https://www.lcsc.com/product-detail/Chip-Resistor-Surface-M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 -> C2889850; LCSC Part Number C2933950 -> (none); LCSC URL (none) -> https://www.lcsc.com/product-detail/Chip-Resistor-Surface-M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
- R7: LCSC https://www.lcsc.com/product-detail/Chip-Resistor-Surface-M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 -> C407275; LCSC Part Number C407275 -> (none); LCSC URL (none) -> https://www.lcsc.com/product-detail/Chip-Resistor-Surface-M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
- U1: LCSC https://www.lcsc.com/product-detail/Charge-Pumps_RENESAS-IC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 -> C7881; LCSC Part Number C7881 -> (none); LCSC URL (none) -> https://www.lcsc.com/product-detail/Charge-Pumps_RENESAS-IC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
- U3: LCSC https://www.lcsc.com/product-detail/Operational-Amplifier_T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 -> C7950; LCSC Part Number C5423 -> (none); LCSC URL (none) -> https://www.lcsc.com/product-detail/Operational-Amplifier_T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
- U4: LCSC https://www.lcsc.com/product-detail/Microcontrollers-MCU-MP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 -> C8734; LCSC Part Number C8734 -> (none); LCSC URL (none) -> https://www.lcsc.com/product-detail/Microcontrollers-MCU-MP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
- U6: LCSC https://www.lcsc.com/product-detail/Voltage-Regulators-Line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 -> C347222; LCSC Part Number C347222 -> (none); LCSC URL (none) -> https://www.lcsc.com/product-detail/Voltage-Regulators-Line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
- U7, U8, U9: LCSC https://www.lcsc.com/product-detail/Operational-Amplifier_T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 -> C1347395; LCSC Part Number C1347395 -> (none); LCSC URL (none) -> https://www.lcsc.com/product-detail/Operational-Amplifier_T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
- Y1: LCSC https://www.lcsc.com/product-detail/Crystals_Seiko-Epson-Q1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 -> C16320; LCSC Part Number C16320 -> (none); LCSC URL (none) -> https://www.lcsc.com/product-detail/Crystals_Seiko-Epson-Q1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
- Y2: LCSC https://www.lcsc.com/product-detail/Crystals_YXC-Crystal-Os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 -> C12674; LCSC Part Number C12674 -> (none); LCSC URL (none) -> https://www.lcsc.com/product-detail/Crystals_YXC-Crystal-Os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
Connections:
- net usb_N is gone; now on net USB_D-: J1.2 (D-)
- net usb_P is gone; now on net USB_D+: J1.3 (D+)
- net +3.3V: now also R40.1
- net +5VA: now also C33.2, C35.2, C37.2
- net -5VA: now also C34.1, C36.1, C38.1
- net GNDA: now also C33.1, C34.2, C35.1, C36.2, C37.1, C38.2
- net HT_Drive_Pulse: now also R40.2
- net HT_Power: now also Q8.3 (D)
- net Peak_Reset: now also R23.1; no longer R23.2
- net at Q3.2 (B), Q6.1 (C), U8.6: no longer R20.2
- net at C16.1, C4.1, C5.1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: now also R37.2, Q8.2 (S); no longer R37.1
- net at Q1.1 (G), Q2.1 (C): now also R37.1; no longer R37.2
- net at C13.2, R29.1: now also Q8.1 (G)
- net at Q6.2 (B): now also R23.2; no longer R23.1
- net at C8.2, Q3.3 (E), Q5.1 (C)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: now also R20.2
Other:
- note added: "MCU"
- note added: "Mounting holes, graphics"
- moved on the sheet: C17, C19, C20, C21, C22, C23, C24, C25, C26, C27, C28, C29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
