File: ScintillatorProbeHardware_v2/HT_Source.kicad_sch (KiCad schematic)
At the start: 36 parts

Commit message: some work
Parts:
- removed C?: 1u, Capacitor_SMD:C_0603_1608Metric, symbol Device:C
- removed Q?: MDD2302, Package_TO_SOT_SMD:SOT-23, symbol Device:Q_NMOS_GSD
- removed R?: 47R, Resistor_SMD:R_0805_2012Metric, symbol Device:R
- removed R?: 100k, Resistor_SMD:R_0603_1608Metric, symbol Device:R
Connections:
- net Power: now reaches C?.1, C?.1, C?.1, R?.2, T?.1 (AA)
- net HT_Drive_Pulse renamed Drive_Pulse
- net HT_Sense renamed Sense
Other:
- moved on the sheet: C?, D?, R?, U?A
