File: ScintillatorProbeHardware_v2/MCU.kicad_sch (KiCad schematic)
At the start: 1 part, among them U1 STM32H723ZGTx

Commit message: some work
Parts:
- added C?: 100n, Capacitor_SMD:C_0603_1608Metric, symbol Device:C
- added J?: Conn_01x02, Connector_PinHeader_2.54mm:PinHeader_1x02_P2.54mm_Vertical, symbol Connector_Generic:Conn_01x02
- added R?: 10k, Resistor_SMD:R_0603_1608Metric, symbol Device:R
- renumbered U1 to U?
Connections:
- net GND: now reaches U?.107 (VSS), U?.120 (VSS), U?.130 (VSS), U?.16 (VSS), U?.38 (VSS), U?.51 (VSS), U?.61 (VSS), U?.83 (VSS), U?.94 (VSS)
- net GND: now also C?.1, J?.1 (Pin_1)
- net +3.3V: now reaches U?.108 (VDD)
- net +3.3V: now also U?.121 (VDD), U?.131 (VDD), U?.144 (VDD), U?.17 (VDD), U?.30 (VDD), U?.39 (VDD), U?.52 (VDD), U?.62 (VDD), U?.72 (VDD), U?.84 (VDD), U?.95 (VDD33USB), R?.2
- net at U?.25 (NRST): now also C?.2, J?.2 (Pin_2), R?.1
- net GNDA: now reaches U?.31 (VSSA)
- net +3.3VA: now reaches U?.33 (VDDA)
