File: ScintillatorProbeHardware_v2/Power.kicad_sch (KiCad schematic)
At the start: 0 parts

Commit message: some work
Parts:
- added C? (x4): 10u, Capacitor_SMD:CP_Elec_4x5.4, symbol Device:C_Polarized
- added C?: 100n, Capacitor_SMD:C_0603_1608Metric, symbol Device:C
- added FB? (x3): 620Ω@1MHz, Inductor_SMD:L_1210_3225Metric, symbol Device:FerriteBead
- added U?: ICL7660, Package_SO:SOIC-8_3.9x4.9mm_P1.27mm, symbol Regulator_SwitchedCapacitor:ICL7660
- added U?: LM358, Package_SO:SOIC-8_3.9x4.9mm_P1.27mm, symbol Amplifier_Operational:LM358
Connections:
- new net: C?.1, U?.2 (CAP+)
- new net: C?.2, U?.4 (CAP-)
- new net +5V: FB?.1, U?.8 (V+)
- new net +5VA: C?.1, C?.2, FB?.2, U?.8 (V+)
- new net -5V: C?.2, FB?.1, U?.5 (VOUT)
- new net -5VA: C?.1, C?.2, FB?.2, U?.4 (V-)
- new net GND: C?.1, FB?.1, U?.3 (GND)
- new net GNDA: C?.1, C?.2, FB?.2
