File: ScintillatorProbeHardware_v2/ScintillatorProbeHardware_v2.kicad_sch (KiCad schematic)
At the start: 0 parts

Commit message: some work
Other:
- added sheet Peak_Detector (Peak_Detector.kicad_sch)
- sheet HT_Source ports: added Drive_Pulse, HT, Power, Sense; removed none
- sheet Power ports: added none; removed 12V, 3V3, USB_5V
- sheet USB ports: added none; removed USB_5V
Changed lines of the file:
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@@
+			)
+		)
+		(pin "Power" input
+			(at 116.84 102.87 180)
+			(effects
+				(font
+					(size 1.27 1.27)
+				)
+				(justify left)
+			)
+		)
+		(pin "Drive_Pulse" input
+			(at 116.84 105.41 180)
+			(effects
+				(font
+					(size 1.27 1.27)
+				)
+				(justify left)
+			)
+		)
+		(pin "Sense" output
+			(at 116.84 107.95 180)
+			(effects
+				(font
+					(size 1.27 1.27)
+				)
+				(justify left)
+			)
+		)
+		(pin "HT" output
+			(at 137.16 104.14 0)
+			(effects
+				(font
+					(size 1.27 1.27)
+				)
+				(justify right)
 			)
 		)
@@
 			)
 		)
-		(pin "USB_5V" output
-			(at 91.44 83.82 0)
-			(effects
-				(font
-					(size 1.27 1.27)
-				)
-				(justify right)
-			)
-		)
 		(instances
 			(project "ScintillatorProbeHardware_v2"
@@
 			)
 		)
-		(pin "USB_5V" input
-			(at 91.44 99.06 0)
-			(effects
-				(font
-					(size 1.27 1.27)
-				)
-				(justify right)
-			)
-		)
-		(pin "12V" output
-			(at 91.44 102.87 0)
-			(effects
-				(font
-					(size 1.27 1.27)
-				)
-				(justify right)
-			)
-		)
-		(pin "3V3" output
-			(at 91.44 106.68 0)
-			(effects
-				(font
-					(size 1.27 1.27)
-				)
-				(justify right)
-			)
-		)
 		(instances
 			(project "ScintillatorProbeHardware_v2"
@@
 				)
 			)
+		)
+	)
+	(sheet
+		(at 151.13 66.04)
+		(size 21.59 21.59)
+		(exclude_from_sim no)
+		(in_bom yes)
+		(on_board yes)
+		(dnp no)
+		(fields_autoplaced yes)
+		(stroke
+			(width 0.1524)
+			(type solid)
+		)
+		(fill
+			(color 0 0 0 0.0000)
+		)
+		(property "Sheetname" "Peak_Detector"
+			(at 151.13 65.3284 0)
+			(effects
+				(font
+					(size 1.27 1.27)
+				)
+				(justify left bottom)
+			)
+		)
+		(property "Sheetfile" "Peak_Detector.kicad_sch"
+			(at 151.13 88.2146 0)
+			(effects
+				(font
+					(size 1.27 1.27)
+				)
+				(justify left top)
+			)
+		)
+		(instances
+			(project "ScintillatorProbeHardware_v2"
+				(path "/736f2e97-1393-4b3c-b920-d97e4221d830"
+					(page "6")
+				)
+			)
