File: ScintillatorProbeHardware_v2/USB.kicad_sch (KiCad schematic)
At the start: 0 parts

Commit message: some work
Parts:
- added J?: USB_B, CustomParts:Amphenol_USB_B, symbol Connector:USB_B
Connections:
- net USB_N: now also J?.2 (D-)
- net USB_P: now also J?.3 (D+)
- new net +5V: J?.1 (VBUS)
- new net GND: J?.4 (GND), J?.5 (Shield)
